File: kicad/88MPH.kicad_pcb (KiCad board)
At the start: 2 copper layers, 102.9 x 31.8 mm, 27 parts, among them CON1 AVR-ISP-6, IC1 ATMEGA328P-P, P1 CONN_01X04, Q1 Q_NPN_EBC, Q2 Q_NPN_EBC

Commit message: Fixed cathode pin 3
Connections:
- D1 pad 3: CK -> CK1
- D2 pad 3: CK -> CK2
Routing:
- net CK2: track 44.7 -> 54.6 mm, vias 0 -> 1
- net CK1: track 74.5 -> 81.0 mm
